Commit message: Manually added mass to links that were missing it

File: robots/blue_left_v2.urdf (robot description, URDF)
Before this commit: robot blue_descriptions_left, 18 links, 17 joints
Links:
- link base_link: mass None -> 0
- link left_elbow_accel_link: mass None -> 0
- link left_gripper_finger_link: mass None -> 0
- link left_shoulder_accel_link: mass None -> 0
- link left_wrist_accel_link: mass None -> 0
